File: audio.kicad_sch (KiCad schematic)
At the start: 41 parts, among them J13 SpeakerL, J14 SpeakerR, J4 SJ1-3525N, U6 NC7WV16P6X, U7 PAM8302AAD, U8 PAM8302AAD

Commit message: update layout pcb & zip tesi
Parts:
- added D6: BAV99, Package_TO_SOT_SMD:SOT-23, symbol Diode:BAV99
Connections:
- net +5V: now also D6.2 (A)
- net GND: now also D6.1 (K); no longer J4.1
- new net: D6.3 (K), J4.1
Other:
- moved on the sheet: J13, J14
Changed lines of the file:
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@@
 	(wire
 		(pts
-			(xy 123.825 121.285) (xy 126.365 121.285)
+			(xy 158.115 114.3) (xy 158.115 118.11)
+		)
+		(stroke
+			(width 0)
+			(type default)
+		)
+	)
+	(wire
+		(pts
+			(xy 123.825 120.65) (xy 126.365 120.65)
 		)
 		(stroke
@@
 	(wire
 		(pts
-			(xy 123.825 108.585) (xy 123.825 121.285)
+			(xy 123.825 108.585) (xy 123.825 120.65)
 		)
 		(stroke
@@
 	(wire
 		(pts
-			(xy 121.92 154.94) (xy 127 154.94)
+			(xy 121.92 151.13) (xy 126.365 151.13)
 		)
 		(stroke
@@
 	(wire
 		(pts
-			(xy 121.92 140.97) (xy 121.92 154.94)
-		)
-		(stroke
-			(width 0)
-			(type default)
-		)
-	)
-	(wire
-		(pts
 			(xy 34.29 96.52) (xy 34.29 89.535)
 		)
@@
 	(wire
 		(pts
+			(xy 121.92 140.97) (xy 121.92 151.13)
+		)
+		(stroke
+			(width 0)
+			(type default)
+		)
+	)
+	(wire
+		(pts
 			(xy 83.82 108.585) (xy 86.995 108.585)
 		)
@@
 	(wire
 		(pts
+			(xy 109.855 153.67) (xy 109.855 157.48)
+		)
+		(stroke
+			(width 0)
+			(type default)
+		)
+	)
+	(wire
+		(pts
 			(xy 68.58 85.09) (xy 68.58 93.345)
 		)
@@
 	(wire
 		(pts
-			(xy 119.38 135.89) (xy 119.38 118.745)
+			(xy 119.38 135.89) (xy 119.38 118.11)
 		)
 		(stroke
@@
 	(wire
 		(pts
-			(xy 127 157.48) (xy 109.855 157.48)
+			(xy 126.365 153.67) (xy 109.855 153.67)
 		)
 		(stroke
@@
 	(wire
 		(pts
-			(xy 119.38 118.745) (xy 126.365 118.745)
+			(xy 119.38 118.11) (xy 126.365 118.11)
 		)
 		(stroke
@@
 	(wire
 		(pts
-			(xy 121.92 125.73) (xy 146.685 125.73)
+			(xy 121.92 125.73) (xy 153.035 125.73)
 		)
 		(stroke
@@
 	(wire
 		(pts
+			(xy 158.115 137.16) (xy 158.115 133.35)
+		)
+		(stroke
+			(width 0)
+			(type default)
+		)
+	)
+	(wire
+		(pts
 			(xy 38.1 100.33) (xy 40.64 100.33)
 		)
@@
 	(global_label "+5V"
 		(shape input)
+		(at 158.115 114.3 180)
+		(fields_autoplaced yes)
+		(effects
+			(font
+				(size 1.27 1.27)
+			)
+			(justify right)
+		)
+		(property "Intersheetrefs" "${INTERSHEET_REFS}"
+			(at 151.2593 114.3 0)
+			(effects
+				(font
+					(size 1.27 1.27)
+				)
+				(justify right)
+				(hide yes)
+			)
+		)
+	)
+	(global_label "+5V"
+		(shape input)
 		(at 68.58 81.915 180)
 		(fields_autoplaced yes)
@@
 	)
 	(symbol
+		(lib_id "Diode:BAV99")
+		(at 158.115 125.73 270)
+		(mirror x)
+		(unit 1)
+		(exclude_from_sim no)
+		(in_bom yes)
+		(on_board yes)
+		(dnp no)
+		(property "Reference" "D6"
+			(at 160.1216 126.9422 90)
+			(effects
+				(font
+					(size 1.27 1.27)
+				)
+				(justify left)
+			)
+		)
+		(property "Value" "BAV99"
+			(at 160.1216 124.5179 90)
+			(effects
+				(font
+					(size 1.27 1.27)
+				)
+				(justify left)
+			)
+		)
+		(property "Footprint" "Package_TO_SOT_SMD:SOT-23"
+			(at 145.415 125.73 0)
+			(effects
+				(font
+					(size 1.27 1.27)
+				)
+				(hide yes)
+			)
+		)
+		(property "Datasheet" "https://assets.nexperia.com/documents/data-sheet/BAV99_SER.pdf"
+			(at 158.115 125.73 0)
+			(effects
+				(font
+					(size 1.27 1.27)
+				)
+				(hide yes)
+			)
+		)
+		(property "Description" "BAV99 High-speed switching diodes, SOT-23"
+			(at 158.115 125.73 0)
+			(effects
+				(font
+					(size 1.27 1.27)
+				)
+				(hide yes)
+			)
+		)
+		(pin "2"
+		)
+		(pin "3"
+		)
+		(pin "1"
+		)
+		(instances
+			(project "Board Console 2023"
+				(path "/306f3bb0-3e7b-4e83-a527-90f1c0ddb0d4/3caec7dc-570b-44e3-af56-bafd59850fb7"
+					(reference "D6")
+					(unit 1)
+				)
+			)
+		)
+	)
+	(symbol
 		(lib_id "Connector_Generic:Conn_01x02")
-		(at 132.08 154.94 0)
+		(at 131.445 151.13 0)
 		(unit 1)
 		(exclude_from_sim no)
@@
 		(fields_autoplaced yes)
 		(property "Reference" "J14"
-			(at 134.112 154.9978 0)
+			(at 133.477 151.1878 0)
 			(effects
 				(font
@@
 		)
 		(property "Value" "SpeakerR"
-			(at 134.112 157.4221 0)
+			(at 133.477 153.6121 0)
 			(effects
 				(font
@@
 		)
 		(property "Footprint" "Connector_PinHeader_2.54mm:PinHeader_1x02_P2.54mm_Vertical"
-			(at 132.08 154.94 0)
+			(at 131.445 151.13 0)
 			(effects
 				(font
@@
 		)
 		(property "Datasheet" "~"
-			(at 132.08 154.94 0)
+			(at 131.445 151.13 0)
 			(effects
 				(font
@@
 		)
 		(property "Description" "Generic connector, single row, 01x02, script generated (kicad-library-utils/schlib/autogen/connector/)"
-			(at 132.08 154.94 0)
+			(at 131.445 151.13 0)
 			(effects
 				(font
@@
 	(symbol
 		(lib_id "power:GND")
-		(at 146.685 125.73 0)
+		(at 158.115 137.16 0)
 		(unit 1)
 		(exclude_from_sim no)
@@
 		(fields_autoplaced yes)
 		(property "Reference" "#PWR037"
-			(at 146.685 132.08 0)
+			(at 158.115 143.51 0)
 			(effects
 				(font
@@
 		)
 		(property "Value" "GND"
-			(at 146.685 129.8631 0)
+			(at 158.115 141.2931 0)
 			(effects
 				(font
@@
 		)
 		(property "Footprint" ""
-			(at 146.685 125.73 0)
+			(at 158.115 137.16 0)
 			(effects
 				(font
@@
 		)
 		(property "Datasheet" ""
-			(at 146.685 125.73 0)
+			(at 158.115 137.16 0)
 			(effects
 				(font
@@
 		)
 		(property "Description" "Power symbol creates a global label with name \"GND\" , ground"
-			(at 146.685 125.73 0)
+			(at 158.115 137.16 0)
 			(effects
 				(font
@@
 	(symbol
 		(lib_id "Connector_Generic:Conn_01x02")
-		(at 131.445 118.745 0)
+		(at 131.445 118.11 0)
 		(unit 1)
 		(exclude_from_sim no)
@@
 		(fields_autoplaced yes)
 		(property "Reference" "J13"
-			(at 133.477 118.8028 0)
+			(at 133.477 118.1678 0)
 			(effects
 				(font
@@
 		)
 		(property "Value" "SpeakerL"
-			(at 133.477 121.2271 0)
+			(at 133.477 120.5921 0)
 			(effects
 				(font
@@
 		)
 		(property "Footprint" "Connector_PinHeader_2.54mm:PinHeader_1x02_P2.54mm_Vertical"
-			(at 131.445 118.745 0)
+			(at 131.445 118.11 0)
 			(effects
 				(font
@@
 		)
 		(property "Datasheet" "~"
-			(at 131.445 118.745 0)
+			(at 131.445 118.11 0)
 			(effects
 				(font
@@
 		)
 		(property "Description" "Generic connector, single row, 01x02, script generated (kicad-library-utils/schlib/autogen/connector/)"
-			(at 131.445 118.745 0)
+			(at 131.445 118.11 0)
 			(effects
 				(font
